Commit message: body.dae

File: eklavya_description/urdf/gazebo.urdf.xacro (robot description, xacro)
@@ -26,5 +26,5 @@
 	  <insert_block name="origin" />
      <geometry>
-     <mesh filename="package://eklavya_description/meshes/body1.dae" />
+     <mesh filename="package://eklavya_description/meshes/body.dae" />
       <!--   <box size="${base_x_size} ${base_y_size} ${base_z_size}" />  -->
   	 <!-- <insert_block name="box" /> -->
