Commit message: orientation fixed

File: eklavya_description/urdf/eklavya_castor.xacro (robot description, xacro)
@@ -7,5 +7,5 @@
  <macro name="caster_support_hinge" params="suffix parent">
 	<joint name="${parent}_caster_support_hinge_${suffix}_joint" type="continuous">
-      <origin  rpy="0 0 0" xyz="${+base_x_size/2 -wheelhub_x_size/2} 0 ${castor_x_size/2 -wheel_x_size/2 -base_z_origin_to_caster_wheel_origin}"/>
+      <origin  rpy="0 0 0" xyz="${-base_x_size/2 +wheelhub_x_size/2} 0 ${castor_x_size/2 -wheel_x_size/2 -base_z_origin_to_caster_wheel_origin}"/>
       <parent link="${parent}" />
       <child link="${parent}_caster_support_hinge_${suffix}_link"/>

File: eklavya_description/urdf/params.xacro (robot description, xacro)
@@ -19,5 +19,5 @@
 	<property name="wheel_y_size" value="0.22000000" />
 	<property name="wheel_z_size" value="0.09000000" />
-	<property name="base_x_origin_to_wheel_origin" value="-0.16" />
+	<property name="base_x_origin_to_wheel_origin" value="0.16" />
 	<property name="base_y_origin_to_wheel_origin" value="0.220" />
 	<property name="base_z_origin_to_wheel_origin" value="0" />
