Commit message: model better

File: eklavya_description/urdf/eklavya_body.urdf.xacro (robot description, xacro)
@@ -67,9 +67,9 @@
     <gazebo_eklavya_base_link_surface />
 	 <!-- WHEEL macros -->
-    <eklavya_wheel suffix="left" parent="base_link">
-      <origin xyz="${-1*base_x_origin_to_wheel_origin} ${-1*base_y_origin_to_wheel_origin} ${ -1*base_z_origin_to_wheel_origin}" rpy="${M_PI} 0 0" />
+  <eklavya_wheel suffix="left" parent="base_link">
+      <origin xyz="${base_x_origin_to_wheel_origin} ${-1*base_y_origin_to_wheel_origin} ${ -1*base_z_origin_to_wheel_origin}" rpy="0 0 0" />
     </eklavya_wheel>
     <eklavya_wheel suffix="right" parent="base_link">
-      <origin xyz="${-1*base_x_origin_to_wheel_origin} ${base_y_origin_to_wheel_origin} ${ -1*base_z_origin_to_wheel_origin}" rpy="0 0 0" />
+      <origin xyz="${base_x_origin_to_wheel_origin} ${base_y_origin_to_wheel_origin} ${ -1*base_z_origin_to_wheel_origin}" rpy="0 0 0" />
     </eklavya_wheel>
     <!-- Castor -->
@@ -77,23 +77,23 @@
     <caster_wheel suffix="front" parent="base_link" />
 	<!-- Controllers -->
-	<!--<gazebo_eklavya_simple_drive_plugin />-->
+	 <gazebo_eklavya_simple_drive_plugin />
 	<!--<gazebo_eklavya_drive_plugin /> -->
-	   <gazebo_eklavya_drive_plugin_diffdrive />  <!-- cmd_vel movement -->
-	 <!-- <gazebo_eklavya_p3d_plugin />--> <!-- Ground Truth-->
-	 <!-- <eklavya_controllers_common /> -->
+	<!--  <gazebo_eklavya_drive_plugin_diffdrive />-->  <!-- cmd_vel movement -->
+	   <gazebo_eklavya_p3d_plugin />  <!-- Ground Truth-->
+	 <eklavya_controllers_common />
     <!-- Simulation sensors -->
-   <!-- <hokuyo_urg name="hokuyo_laser" parent="base_link" >
-      <origin rpy="0 0 ${M_PI}" xyz="${-base_x_size/2} 0  0.33"/>
-    </hokuyo_urg> -->
+    <hokuyo_urg name="hokuyo_laser" parent="base_link" >
+      <origin rpy="0 0 0" xyz="${base_x_size/2} 0  ${base_z_size-0.03}"/>
+    </hokuyo_urg>
 	<!--<sick_lms100_200 name="sick_laser" parent="base_link" >
 		<origin rpy="0 0 0" xyz="${base_x_size/2+0.12} 0  0.080"/>
 	</sick_lms100_200>   -->
-	<!-- <microstrain_imu name="eklavya_sim_imu" parent="base_link" imu_topic="imu/data" update_rate="30" stdevNoise="0.0017">
+	  <microstrain_imu name="eklavya_sim_imu" parent="base_link" imu_topic="imu/data" update_rate="30" stdevNoise="0.0017">
 		 <origin rpy="0 0 0" xyz="0 0 0"/>
-	</microstrain_imu> -->
+	</microstrain_imu>
     <!-- Kinect frames and mounting (includes simulation) -->
-   <!-- <eklavya_kinect> -->
+     <eklavya_kinect>
 	  <!--origin rpy="0 0 ${M_PI/2}" xyz="${-base_x_size/2-0.05} 0  0.6"/-->
-	<!--</eklavya_kinect> -->
+	 </eklavya_kinect>
   </xacro:macro>
 </robot>

File: eklavya_description/urdf/eklavya_calibration.xacro (robot description, xacro)
@@ -1,10 +1,10 @@
 <?xml version="1.0"?>
 <robot>
-  <property name="eklavya_calib_cam_x" value="${-0.0844382+0.36-0.55}" />
+  <property name="eklavya_calib_cam_x" value="${-0.0844382+base_x_size/4}" />
   <property name="eklavya_calib_cam_y" value="${0+ 0}" />
-  <property name="eklavya_calib_cam_z" value="${0.05+0.55-0.18}" />
+  <property name="eklavya_calib_cam_z" value="${cam_pole+base_z_size}" />
   <property name="eklavya_calib_cam_rr" value="0" />
-  <property name="eklavya_calib_cam_rp" value="0" />
-  <property name="eklavya_calib_cam_ry" value="3.1415926535897932384626" />
+  <property name="eklavya_calib_cam_rp" value="${cam_angle}" />
+  <property name="eklavya_calib_cam_ry" value="0" />
   <property name="eklavya_camera_parent_name" value="base_link" />
 </robot>

File: eklavya_description/urdf/eklavya_hardware.xacro (robot description, xacro)
@@ -7,5 +7,5 @@
  <macro name="caster_support_hinge" params="suffix parent">
 	<joint name="${parent}_caster_support_hinge_${suffix}_joint" type="continuous">
-      <origin  rpy="0 0 ${M_PI}" xyz="${-base_x_size/2 +wheelhub_x_size/2} 0 ${castor_x_size/2 -wheel_x_size/2 -base_z_origin_to_caster_wheel_origin}"/>
+      <origin  rpy="0 0 ${M_PI}" xyz="${+base_x_size/2 -wheelhub_x_size/2} 0 ${castor_x_size/2 -wheel_x_size/2 -base_z_origin_to_caster_wheel_origin}"/>
       <parent link="${parent}" />
       <child link="${parent}_caster_support_hinge_${suffix}_link"/>

File: eklavya_description/urdf/eklavya_wheel.xacro (robot description, xacro)
@@ -5,5 +5,5 @@
   xmlns:interface="http://playerstage.sourceforge.net/gazebo/xmlschema/#interface">
     <include filename="$(find eklavya_description)/urdf/params.xacro"/>
-	<property name="wheel_mass" value="2.63657000" /> <!-- in kg-->
+	<property name="wheel_mass" value="2.6" /> <!-- in kg-->
   <macro name="eklavya_wheel" params="suffix parent *origin">
     <joint name="${parent}_${suffix}_wheel_joint" type="continuous">
@@ -35,5 +35,5 @@
       <joint name="${parent}_${suffix}_wheel_joint" />
       <mechanicalReduction>1.0</mechanicalReduction>
-      <motorTorqueConstant>1</motorTorqueConstant>
+       <!-- <motorTorqueConstant>1</motorTorqueConstant>-->
     </transmission>
   </macro>

File: eklavya_description/urdf/gazebo.urdf.xacro (robot description, xacro)
@@ -26,5 +26,5 @@
 	  <insert_block name="origin" />
      <geometry>
-     <mesh filename="package://eklavya_description/meshes/body.dae" />
+     <mesh filename="package://eklavya_description/meshes/body1.dae" />
       <!--   <box size="${base_x_size} ${base_y_size} ${base_z_size}" />  -->
   	 <!-- <insert_block name="box" /> -->
@@ -33,5 +33,5 @@
   </macro>
   <macro name="eklavya_castor_support_link_mesh">
-    <origin xyz="0 0 0" rpy="0 0 ${M_PI}" />
+    <origin xyz="0 0 0" rpy="0 0 0" />
     <geometry>
       <mesh filename="package://eklavya_description/meshes/wheelhub.dae"/>
@@ -41,5 +41,5 @@
   </macro>
   <macro name="eklavya_castor_wheel_link_mesh">
-	  <origin xyz="0 0 0" rpy="1.570796327 0 0" />
+	  <origin xyz="0 0 0" rpy="${M_PI/2} 0 0" />
     <!--<origin xyz="0 0 0" rpy="0 0 0" /> -->
     <geometry>
@@ -49,5 +49,5 @@
   </macro>
  <macro name="eklavya_wheel_mesh" params="suffix">
-    <origin xyz="0 0 0" rpy="1.570796327 0 0" />
+    <origin xyz="0 0 0" rpy="${M_PI/2} 0 0" />
     <geometry>
       <mesh filename="package://eklavya_description/meshes/wheel.dae" />
@@ -91,5 +91,5 @@
     <leftJoint>base_link_left_wheel_joint</leftJoint>
     <rightJoint>base_link_right_wheel_joint</rightJoint>
-    <wheelSeparation>${base_y_size}</wheelSeparation>
+    <wheelSeparation>${base_y_origin_to_wheel_origin*2}</wheelSeparation>
     <wheelDiameter>${wheel_x_size/2}</wheelDiameter>
     <torque>30</torque>
@@ -119,5 +119,5 @@
                 <leftJoint>base_link_left_wheel_joint</leftJoint>
                 <rightJoint>base_link_right_wheel_joint</rightJoint>
-                <wheelSeparation>${base_y_size}</wheelSeparation>
+                <wheelSeparation>${base_y_origin_to_wheel_origin*2}</wheelSeparation>
                 <wheelDiameter>${wheel_x_size}</wheelDiameter>
                 <torque>20</torque>

File: eklavya_description/urdf/hokuyo_urg.xacro (robot description, xacro)
@@ -18,5 +18,5 @@
             </inertial>
             <visual>
-                <origin xyz="0.0 0.0 0.0" rpy="${M_PI/2} 0 ${M_PI/2}" />
+                <origin xyz="0 0 0" rpy="${M_PI/2} 0 ${M_PI/2}" />
                 <geometry>
                     <mesh filename="package://eklavya_description/meshes/collada/hokuyo_urg.dae"/>
@@ -25,5 +25,5 @@
             </visual>
             <collision>
-                <origin xyz="0.0 0.0 0.0" rpy="${M_PI/2} 0 ${M_PI/2}" />
+                <origin xyz="0 0 0" rpy="${M_PI/2} 0 ${M_PI/2}" />
                 <geometry>
                     <mesh filename="package://eklavya_description/meshes/collada/hokuyo_urg.dae"/>

File: eklavya_description/urdf/params.xacro (robot description, xacro)
@@ -22,5 +22,5 @@
 	<property name="base_y_origin_to_wheel_origin" value="0.220" />
 	<property name="base_z_origin_to_wheel_origin" value="0" />
-	<property name="base_x_origin_to_caster_wheel_origin" value="-0.068" />
+	<property name="base_x_origin_to_caster_wheel_origin" value="0.068" />
 	<property name="base_y_origin_to_caster_wheel_origin" value="0.0" />
 	<property name="base_z_origin_to_caster_wheel_origin" value="-0.085" />
@@ -32,3 +32,5 @@
 	<property name="wheelhub_z_size" value="0.12000000" />
 	<property name="caster_support_hinge_z_offset" value="0.0325" /> <!-- 0.06275 0.05325 .058-->
+	<property name="cam_pole" value="0.22" />
+    <property name="cam_angle" value="${M_PI/8}" />
 </robot>

Commit message: Fixed model

File: eklavya_description/urdf/eklavya_body.urdf.xacro (robot description, xacro)
@@ -8,5 +8,5 @@
   <include filename="$(find eklavya_description)/urdf/gazebo.urdf.xacro"/>
   <include filename="$(find eklavya_description)/urdf/materials.urdf.xacro"/>
-  <include filename="$(find eklavya_description)/urdf/eklavya_hardware.xacro"/>
+  <include filename="$(find eklavya_description)/urdf/eklavya_castor.xacro"/>
   <include filename="$(find eklavya_description)/urdf/eklavya_wheel.xacro"/>
   <include filename="$(find eklavya_description)/urdf/hokuyo_urg.xacro"/>
@@ -18,48 +18,47 @@
     <!-- BASE-FOOTPRINT -->
     <!-- base_footprint is a fictitious link(frame) that is on the ground right below base_link origin, navigation stack depends on this frame -->
-    <link name="base_footprint">
-      <visual>
-        <origin xyz="0 0 0" rpy="0 0 0" />
-        <geometry>
-          <box size="0.1 0.1 0.01" />
-        </geometry>
-      </visual>
-      <inertial>
-            <mass value="0.0001" />
-            <origin xyz="0 0 0" />
-            <inertia ixx="0.0001" ixy="0.0" ixz="0.0"
-                iyy="0.0001" iyz="0.0"
-                izz="0.0001" />
-        </inertial>
-	<!--  <collision>
-          <origin xyz="0 0 0.0" rpy="0 0 0" />
-          <geometry>
-            <box size="0.001 0.001 0.001" />
-         </geometry>
-      </collision>-->
-    </link>
-    <gazebo reference="base_footprint">
-        <material>Gazebo/Green</material>
-        <turnGravityOff>false</turnGravityOff>
-    </gazebo>
-    <joint name="base_footprint_joint" type="fixed">
-      <origin xyz="0 0 ${wheel_x_size/2 - base_z_origin_to_wheel_origin}" rpy="0 0 0" />
-      <parent link="base_footprint"/>
-      <child link="base_link" />
-    </joint>
+    <!-- base_footprint is a fictitious link(frame) that is on the ground right below base_link origin,
+             navigation stack depends on this frame -->
+	<link name="base_footprint">
+		<visual>
+			<origin xyz="0 0 0" rpy="0 0 0" />
+			<geometry>
+				<box size="0.001 0.001 0.001" />
+			</geometry>
+			<material name="Green" />
+		</visual>
+	</link>
+	<joint name="base_footprint_joint" type="fixed">
+		<origin xyz="0 0 0.128" rpy="0 0 0" />
+		<parent link="base_footprint"/>
+		<child link="base_link" />
+	</joint>
     <!-- BASE-LINK -->
     <!--Actual body/chassis of the robot-->
     <link name="base_link">
-	<box_inertial_with_origin x="${base_x_size}" y="${base_y_size}" z="${base_z_size}" mass="${base_mass}" origin="0 0 ${base_z_size/2}" />
+	<!--<box_inertial_with_origin x="${base_x_size}" y="${base_y_size}" z="${base_z_size}" mass="${base_mass}" origin="0 0 ${base_z_size/2}" />
+      -->
+      <inertial>
+		<mass value="${base_mass}" />
+		<origin xyz="0 0 0" />
+		<inertia ixx="1.0" ixy="0.0" ixz="0.0"
+				 iyy="1.0" iyz="0.0"
+				 izz="1.0" />
+       </inertial>
       <visual>
-        <eklavya_base_link_mesh>
+       <!-- <eklavya_base_link_mesh>
            <origin xyz="0 0 ${base_z_size/2}" rpy="0 0 0" />
            <box size="${base_x_size} ${base_y_size} ${base_z_size}" />
-        </eklavya_base_link_mesh>
+        </eklavya_base_link_mesh> -->
+        <origin xyz="0 0 ${base_z_size/2}" rpy="0 0 0" />
+		<geometry>
+			<mesh filename="package://eklavya_description/meshes/body.dae" />
+		</geometry>
       </visual>
       <collision>
          <origin xyz="0 0 ${base_z_size/2}" rpy="0 0 0" />
          <geometry>
-            <box size = "${base_x_size+0.02} ${base_y_size} ${base_z_size+0.02}"/>--> <!--making it slightly bigger in x and z direction-->
+           <!-- <box size = "${base_x_size+0.02} ${base_y_size} ${base_z_size+0.02}"/>--> <!--making it slightly bigger in x and z direction-->
+			<mesh filename="package://eklavya_description/meshes/body.dae" />
          </geometry>
       </collision>
@@ -67,9 +66,9 @@
     <gazebo_eklavya_base_link_surface />
 	 <!-- WHEEL macros -->
-  <eklavya_wheel suffix="left" parent="base_link">
-      <origin xyz="${base_x_origin_to_wheel_origin} ${-1*base_y_origin_to_wheel_origin} ${ -1*base_z_origin_to_wheel_origin}" rpy="0 0 0" />
+    <eklavya_wheel suffix="left" parent="base_link">
+      <origin xyz="${base_x_origin_to_wheel_origin} ${base_y_origin_to_wheel_origin} 0" rpy="0 0 0" />
     </eklavya_wheel>
     <eklavya_wheel suffix="right" parent="base_link">
-      <origin xyz="${base_x_origin_to_wheel_origin} ${base_y_origin_to_wheel_origin} ${ -1*base_z_origin_to_wheel_origin}" rpy="0 0 0" />
+      <origin xyz="${base_x_origin_to_wheel_origin} ${-1*base_y_origin_to_wheel_origin} 0" rpy="0 0 0" />
     </eklavya_wheel>
     <!-- Castor -->
@@ -77,7 +76,7 @@
     <caster_wheel suffix="front" parent="base_link" />
 	<!-- Controllers -->
-	 <gazebo_eklavya_simple_drive_plugin />
+	<!-- <gazebo_eklavya_simple_drive_plugin /> -->
 	<!--<gazebo_eklavya_drive_plugin /> -->
-	<!--  <gazebo_eklavya_drive_plugin_diffdrive />-->  <!-- cmd_vel movement -->
+	  <gazebo_eklavya_drive_plugin_diffdrive />   <!-- cmd_vel movement -->
 	   <gazebo_eklavya_p3d_plugin />  <!-- Ground Truth-->
 	 <eklavya_controllers_common />
@@ -93,7 +92,5 @@
 	</microstrain_imu>
     <!-- Kinect frames and mounting (includes simulation) -->
-     <eklavya_kinect>
-	  <!--origin rpy="0 0 ${M_PI/2}" xyz="${-base_x_size/2-0.05} 0  0.6"/-->
-	 </eklavya_kinect>
+     <eklavya_kinect />
   </xacro:macro>
 </robot>

File: eklavya_description/urdf/eklavya_castor.xacro (robot description, xacro)
@@ -7,5 +7,5 @@
  <macro name="caster_support_hinge" params="suffix parent">
 	<joint name="${parent}_caster_support_hinge_${suffix}_joint" type="continuous">
-      <origin  rpy="0 0 ${M_PI}" xyz="${+base_x_size/2 -wheelhub_x_size/2} 0 ${castor_x_size/2 -wheel_x_size/2 -base_z_origin_to_caster_wheel_origin}"/>
+      <origin  rpy="0 0 0" xyz="${+base_x_size/2 -wheelhub_x_size/2} 0 ${castor_x_size/2 -wheel_x_size/2 -base_z_origin_to_caster_wheel_origin}"/>
       <parent link="${parent}" />
       <child link="${parent}_caster_support_hinge_${suffix}_link"/>
@@ -22,15 +22,16 @@
     <link name="${parent}_caster_support_hinge_${suffix}_link">
       <inertial>
-        <mass value="1"/>
-        <origin xyz="0 0 0"/>
-        <inertia ixx="0.00375" ixy="0.0" ixz="0.0"
-          iyy="0.00375" iyz="0.0"
-          izz="0.00375" />
-      </inertial>
+			<mass value="0.1"/>
+			<origin xyz="0 0 0" />
+			<inertia ixx="0.01" ixy="0.0" ixz="0.0"
+					 iyy="0.01" iyz="0.0"
+					 izz="0.01" />
+		</inertial>
       <visual>
         <eklavya_castor_support_link_mesh />
       </visual>
       <collision>
-        <eklavya_collision_none />
+        <!--<eklavya_collision_none />-->
+        <eklavya_castor_support_link_mesh />
       </collision>
     </link>
@@ -52,14 +53,22 @@
     </transmission>
     <link name="${parent}_caster_wheel_${suffix}_link">
-	<cylinder_inertial_with_origin_wheel radius="${castor_x_size/2}" length="${castor_z_size}" mass="1" origin="0 0 0" />
+	<!--<cylinder_inertial_with_origin_wheel radius="${castor_x_size/2}" length="${castor_z_size}" mass="1" origin="0 0 0" /> -->
+	 <inertial>
+		<mass value="0.1" />
+		<origin xyz="0 0 0" rpy="0 0 0" />
+		<inertia  ixx="0.012411765597" ixy="-0.000711733678" ixz="0.00050272983"
+				  iyy="0.015218160428" iyz="-0.000004273467"
+				  izz="0.011763977943" />
+	</inertial>
       <visual>
         <eklavya_castor_wheel_link_mesh />
       </visual>
       <collision>
-		<origin xyz="0 0 0" rpy="1.570796327 0 0" />
-		<!--<origin xyz="0 0 0" rpy="0 0 0" /> -->
+		<eklavya_castor_wheel_link_mesh />
+		<!--
+		<origin xyz="0 0 0" rpy="${M_PI/2} 0 0" />
 		<geometry>
 			<cylinder radius="${castor_x_size/2}" length="${castor_z_size}"/>
-		</geometry>
+		</geometry> -->
       </collision>
     </link>

File: eklavya_description/urdf/eklavya_wheel.xacro (robot description, xacro)
@@ -17,5 +17,13 @@
     </joint>
     <link name="${parent}_${suffix}_wheel_link">
-      <cylinder_inertial_with_origin_wheel radius="${wheel_x_size/2}" length="${wheel_z_size}" mass="${wheel_mass}" origin="0 0 0" />
+      <!--<cylinder_inertial_with_origin_wheel radius="${wheel_x_size/2}" length="${wheel_z_size}" mass="${wheel_mass}" origin="0 0 0" />
+	  -->
+	  <inertial>
+			<mass value="0.1" />
+			<origin xyz=" 0 0 0 " />
+			<inertia  ixx="0.012411765597" ixy="0.0" ixz="0.0"
+					  iyy="0.015218160428" iyz="0.0"
+					  izz="0.011763977943" />
+		</inertial>
 	  <visual>
         <eklavya_wheel_mesh suffix="${suffix}" />

File: eklavya_description/urdf/gazebo.urdf.xacro (robot description, xacro)
@@ -7,27 +7,25 @@
   <macro name="gazebo_eklavya_base_link_surface">
     <gazebo reference="base_link">
-      <!--<mu1 value="100.0" />
-      <mu2 value="100.0" />
-      <kp  value="1000000.0" />
-      <kd  value="1.0" />-->
-      <!--material name="Eklavya/GunMetalBrushedAluminum   Gazebo/Blue" />-->
+    <!--material name="Gazebo/Blue" />-->
     <!--<material>Eklavya/GunMetalBrushedAluminum</material>-->
+    <material>Eklavya/BlueBrushedAluminum</material>
     </gazebo>
   </macro>
   <macro name="gazebo_eklavya_castor_wheel_link_surface" params="suffix parent">
     <gazebo reference="${parent}_caster_wheel_${suffix}_link">
-      <mu1 value="10.0" />
-      <mu2 value="10.0" />
-      <kp  value="1000000.0" />
-      <kd  value="1.0" />
+		<mu1 value="100.0" />
+		<mu2 value="100.0" />
+		<kp  value="1000000.0" />
+		<kd  value="1.0" />
+		<material>Eklavya/Grey</material>
     </gazebo>
   </macro>
   <macro name="eklavya_base_link_mesh"  params="*origin *box" >
-	  <insert_block name="origin" />
+	 <insert_block name="origin" />
      <geometry>
-     <mesh filename="package://eklavya_description/meshes/body.dae" />
+		<mesh filename="package://eklavya_description/meshes/body.dae" />
       <!--   <box size="${base_x_size} ${base_y_size} ${base_z_size}" />  -->
   	 <!-- <insert_block name="box" /> -->
-    </geometry>
+     </geometry>
      <material name="GunMetalBrushedAluminum"/>
   </macro>
@@ -117,9 +115,9 @@
                 <update>100</update>
                 <updateRate>100.0</updateRate>
-                <leftJoint>base_link_left_wheel_joint</leftJoint>
-                <rightJoint>base_link_right_wheel_joint</rightJoint>
-                <wheelSeparation>${base_y_origin_to_wheel_origin*2}</wheelSeparation>
-                <wheelDiameter>${wheel_x_size}</wheelDiameter>
-                <torque>20</torque>
+                <leftJoint>base_link_right_wheel_joint</leftJoint>
+                <rightJoint>base_link_left_wheel_joint</rightJoint>
+                <wheelSeparation>0.3305</wheelSeparation> <!-- ${base_y_origin_to_wheel_origin*2} 0.3305 -->
+                <wheelDiameter>0.15</wheelDiameter> <!-- ${wheel_x_size} 0.15 -->
+                <torque>5</torque>
                 <interface:position name="position_iface_0"/>
                 <robotNamespace>/</robotNamespace>

Commit message: powerful laser

File: eklavya_description/urdf/eklavya_body.urdf.xacro (robot description, xacro)
@@ -28,4 +28,10 @@
 			<material name="Green" />
 		</visual>
+		<collision>
+		  <origin xyz="0 0 0.128" rpy="0 0 0" />
+		  <geometry>
+		   <box size="0.001 0.001 0.001" />
+		  </geometry>
+		</collision>
 	</link>
 	<joint name="base_footprint_joint" type="fixed">
@@ -76,16 +82,17 @@
     <caster_wheel suffix="front" parent="base_link" />
 	<!-- Controllers -->
+	<gazebo_ros_eklavya_plugin />
 	<!-- <gazebo_eklavya_simple_drive_plugin /> -->
-	<gazebo_eklavya_drive_plugin />
+	<!-- <gazebo_eklavya_drive_plugin /> -->
 	 <!-- <gazebo_eklavya_drive_plugin_diffdrive />  -->  <!-- cmd_vel movement -->
-	   <gazebo_eklavya_p3d_plugin />  <!-- Ground Truth-->
+	 <!-- <gazebo_eklavya_p3d_plugin />  Ground Truth-->
 	 <eklavya_controllers_common />
     <!-- Simulation sensors -->
-    <hokuyo_urg name="hokuyo_laser" parent="base_link" >
+    <!--<hokuyo_urg name="hokuyo_laser" parent="base_link" >
       <origin rpy="0 0 0" xyz="${base_x_size/2} 0  ${base_z_size-0.03}"/>
-    </hokuyo_urg>
-	<!--<sick_lms100_200 name="sick_laser" parent="base_link" >
-		<origin rpy="0 0 0" xyz="${base_x_size/2+0.12} 0  0.080"/>
-	</sick_lms100_200>   -->
+    </hokuyo_urg>  -->
+	<sick_lms100_200 name="sick_laser" parent="base_link" >
+		<origin rpy="0 0 0" xyz="${base_x_size/2} 0  ${base_z_size-0.03}"/>
+	</sick_lms100_200>
 	  <microstrain_imu name="eklavya_sim_imu" parent="base_link" imu_topic="imu/data" update_rate="30" stdevNoise="0.0017">
 		 <origin rpy="0 0 0" xyz="0 0 0"/>

File: eklavya_description/urdf/gazebo.urdf.xacro (robot description, xacro)
@@ -126,4 +126,20 @@
          </gazebo>
     </macro>
+	<macro name="gazebo_ros_eklavya_plugin">
+        <gazebo>
+            <controller:gazebo_ros_eklavya name="gazebo_ros_eklavya_controller" plugin="libgazebo_ros_eklavya.so">
+			  <alwaysOn>true</alwaysOn>
+			  <node_namespace>eklavya_node</node_namespace>
+			  <left_wheel_joint>base_link_right_wheel_joint</left_wheel_joint>
+			  <right_wheel_joint>base_link_left_wheel_joint</right_wheel_joint>
+			  <front_castor_wheel_joint>base_link_caster_wheel_front_joint</front_castor_wheel_joint>
+			  <front_castor_swivel_joint>base_link_caster_support_hinge_front_joint</front_castor_swivel_joint>
+			  <wheel_separation>${base_y_origin_to_wheel_origin*2}</wheel_separation> <!-- ${base_y_origin_to_wheel_origin*2} 0.3305 -->
+			  <wheel_diameter>${wheel_x_size}</wheel_diameter> <!-- ${wheel_x_size} 0.15 -->
+			  <updateRate>40</updateRate>
+			  <torque>20</torque>
+			</controller:gazebo_ros_eklavya>
+         </gazebo>
+    </macro>
 	<macro name="gazebo_eklavya_p3d_plugin">
 		 <gazebo>

File: eklavya_description/urdf/sick_lms100_200.urdf.xacro (robot description, xacro)
@@ -86,5 +86,5 @@
                 <maxAngle> 100</maxAngle>
                 <minRange>0.05</minRange>
-                <maxRange>6.0</maxRange>
+                <maxRange>20.0</maxRange>
                 <resRange>0.001</resRange>
                 <updateRate>25.0</updateRate>

Commit message: TF published... Odometry restructured...

File: eklavya_description/urdf/eklavya_body.urdf.xacro (robot description, xacro)
@@ -42,5 +42,5 @@
     <!-- BASE-LINK -->
     <!--Actual body/chassis of the robot-->
-    <link name="base_link">
+    <link name="base_link" parent="base_footprint">
 	<!--<box_inertial_with_origin x="${base_x_size}" y="${base_y_size}" z="${base_z_size}" mass="${base_mass}" origin="0 0 ${base_z_size/2}" />
       -->
